Commit message: Added camera to robot description

File: src/dd_robot/urdf/dd_robot.xacro (robot description, xacro)
@@ -174,4 +174,32 @@
     <child link="lidar_link"/>
     <origin xyz="0 0 0.205" rpy="0 0 0"/>
+  </joint>
+  <!-- Camera Link -->
+  <link name="camera_link">
+    <visual>
+      <origin xyz="0 0 0" rpy="0 0 0"/>
+      <geometry>
+        <box size="0.05 0.05 0.05"/>
+      </geometry>
+      <material name="black">
+        <color rgba="0 0 0 1"/>
+      </material>
+    </visual>
+    <collision>
+      <origin xyz="0 0 0" rpy="0 0 0"/>
+      <geometry>
+        <box size="0.05 0.05 0.05"/>
+      </geometry>
+    </collision>
+    <inertial>
+      <mass value="0.1"/>
+      <inertia ixx="1e-6" ixy="0" ixz="0" iyy="1e-6" iyz="0" izz="1e-6"/>
+    </inertial>
+  </link>
+  <!-- Joint for Camera -->
+  <joint name="camera_joint" type="fixed">
+    <parent link="base_link"/>
+    <child link="camera_link"/>
+    <origin xyz="0.225 0 0.15" rpy="0 0 0"/>
   </joint>
   <!-- Gazebo plugin for LiDAR -->
@@ -209,3 +237,30 @@
     </sensor>
   </gazebo>
+  <gazebo reference="camera_link">
+    <sensor name="camera" type="camera">
+      <pose>0.025 0 0 0 0 0</pose>
+      <update_rate>30</update_rate>
+      <camera>
+        <horizontal_fov>1.3962634</horizontal_fov>
+        <image>
+          <width>640</width>
+          <height>480</height>
+          <format>R8G8B8</format>
+        </image>
+        <clip>
+          <near>0.1</near>
+          <far>100</far>
+        </clip>
+        <noise>
+          <type>gaussian</type>
+          <mean>0.0</mean>
+          <stddev>0.007</stddev>
+        </noise>
+      </camera>
+      <always_on>true</always_on>
+      <visualize>true</visualize>
+      <topic>/camera/image_raw</topic>
+      <frame_name>camera_link</frame_name>
+    </sensor>
+  </gazebo>
 </robot>

Commit message: Added an extra castor wheel to stabilize the robot Got the robot to teleoperate using the keyboard

File: src/dd_robot/urdf/dd_robot.xacro (robot description, xacro)
@@ -62,4 +62,31 @@
     <origin xyz="${caster_offset_x} 0 -${body_height / 2}" rpy="0 0 0"/>
   </joint>
+  <!-- Caster -->
+  <link name="caster2">
+    <visual>
+      <origin xyz="0 0 0" rpy="0 0 0"/>
+      <geometry>
+        <sphere radius="${caster_radius}"/>
+      </geometry>
+      <material name="darkgray">
+        <color rgba=".2 .2 .2 1"/>
+      </material>
+    </visual>
+    <collision>
+      <origin xyz="0 0 0" rpy="0 0 0"/>
+      <geometry>
+        <sphere radius="${caster_radius}"/>
+      </geometry>
+    </collision>
+    <inertial>
+      <mass value="${caster_mass}"/>
+      <inertia ixx="0.0001" ixy="0.0" ixz="0.0" iyy="0.0001" iyz="0.0" izz="0.0001"/>
+    </inertial>
+  </link>
+  <joint name="joint_caster2" type="fixed">
+    <parent link="base_link"/>
+    <child link="caster2"/>
+    <origin xyz="-${caster_offset_x} 0 -${body_height / 2}" rpy="0 0 0"/>
+  </joint>
   <!-- Right Wheel -->
   <link name="right_wheel">
@@ -139,6 +166,5 @@
       <wheel_radius>${wheel_radius}</wheel_radius>
       <odom_publish>true</odom_publish>
-      <odom_topic>/odom</odom_topic>
-      <cmd_vel_topic>/cmd_vel</cmd_vel_topic>
+      <odom_publish_frequency>1</odom_publish_frequency>
       <max_velocity>5.0</max_velocity>
       <min_velocity>-5.0</min_velocity>

Commit message: Working IMU, Joint State Publisher, and Odometry

File: src/dd_robot/urdf/dd_robot.xacro (robot description, xacro)
@@ -165,10 +165,4 @@
       <wheel_separation>${2 * wheel_offset_y}</wheel_separation>
       <wheel_radius>${wheel_radius}</wheel_radius>
-      <odom_publish>true</odom_publish>
-      <odom_publish_frequency>1</odom_publish_frequency>
-      <max_velocity>5.0</max_velocity>
-      <min_velocity>-5.0</min_velocity>
-      <max_acceleration>20.0</max_acceleration>
-      <min_acceleration>-20.0</min_acceleration>
     </plugin>
   </gazebo>
@@ -178,5 +172,5 @@
       <origin xyz="0 0 0" rpy="0 0 0"/>
       <geometry>
-        <cylinder radius="0.05" length="0.02"/>
+        <cylinder radius="0.05" length="0.08"/>
       </geometry>
       <material name="black">
@@ -187,5 +181,5 @@
       <origin xyz="0 0 0" rpy="0 0 0"/>
       <geometry>
-        <cylinder radius="0.05" length="0.02"/>
+        <cylinder radius="0.05" length="0.08"/>
       </geometry>
     </collision>
@@ -199,5 +193,5 @@
     <parent link="base_link"/>
     <child link="lidar_link"/>
-    <origin xyz="0 0 0.205" rpy="0 0 0"/>
+    <origin xyz="0 0 0.165" rpy="0 0 0"/>
   </joint>
   <!-- Camera Link -->
@@ -233,8 +227,11 @@
     <plugin name="ignition::gazebo::systems::Sensors" filename="libignition-gazebo-sensors-system.so"/>
   </gazebo>
+  <gazebo>
+    <plugin name="ignition::gazebo::systems::JointStatePublisher" filename="libignition-gazebo-joint-state-publisher-system.so"/>
+  </gazebo>
   <!-- Sensor block -->
   <gazebo reference="lidar_link">
     <sensor name="lidar" type="gpu_lidar">
-      <pose>0 0 0 0 0 0</pose>
+      <pose>0 0 0.04 0 0 0</pose>
       <update_rate>10</update_rate>
       <topic>scan</topic>
@@ -290,3 +287,58 @@
     </sensor>
   </gazebo>
+  <!-- Gazebo plugin for IMU -->
+  <gazebo>
+    <plugin name="ignition::gazebo::systems::Imu" filename="libignition-gazebo-imu-system.so"/>
+  </gazebo>
+  <!-- IMU Link -->
+  <link name="imu_link">
+    <visual>
+      <origin xyz="0 0 0" rpy="0 0 0"/>
+      <geometry>
+        <box size="0.05 0.05 0.02"/>
+      </geometry>
+      <material name="black">
+        <color rgba="0 0 0 1"/>
+      </material>
+    </visual>
+    <collision>
+      <origin xyz="0 0 0" rpy="0 0 0"/>
+      <geometry>
+        <box size="0.05 0.05 0.02"/>
+      </geometry>
+    </collision>
+    <inertial>
+      <mass value="0.05"/>
+      <inertia ixx="1e-6" ixy="0" ixz="0" iyy="1e-6" iyz="0" izz="1e-6"/>
+    </inertial>
+  </link>
+  <!-- Joint for IMU -->
+  <joint name="imu_joint" type="fixed">
+    <parent link="base_link"/>
+    <child link="imu_link"/>
+    <origin xyz="0 0 0.215" rpy="0 0 0"/>
+  </joint>
+  <!-- Gazebo plugin for IMU -->
+  <gazebo reference="imu_link">
+    <sensor name="imu_sensor" type="imu">
+      <pose>0 0 0 0 0 0</pose>
+      <topic>/imu</topic>
+      <update_rate>100</update_rate>
+      <always_on>true</always_on>
+      <visualize>true</visualize>
+      <imu>
+        <angular_velocity>
+          <x>true</x>
+          <y>true</y>
+          <z>true</z>
+        </angular_velocity>
+        <linear_acceleration>
+          <x>true</x>
+          <y>true</y>
+          <z>true</z>
+        </linear_acceleration>
+      </imu>
+      <frame_name>imu_link</frame_name>
+    </sensor>
+  </gazebo>
 </robot>
